File: kicad/simulation/simulation.kicad_sch (KiCad schematic)
At the start: 42 parts, among them Q1 CSD19505KCS, Q2 2N2222, Q3 Q_PMOS_DGS, Q4 Q_NMOS_DGS, U1 OPAMP, U2 OPAMP

Commit message: Prep for release to github.
Parts:
- added R14: 2M, symbol Device:R
- added R15: 1M, symbol Device:R
- C2: Spice_Model 1.6 -> 0.01
- D4: Spice_Node_Sequence (none) -> 2 1
- D6: value 6V8 -> 1V8; Spice_Model ZD6V8 -> ZD1V8; Spice_Node_Sequence (none) -> 2 1
- R11: value 1M -> 2M; Spice_Model 1Meg -> 2meg
- R12: value 1M -> 2M; Spice_Model 1meg -> 2meg
- R13: value 270K -> 1M; Spice_Model 270k -> 1Meg
- R18: renamed from R16; value 4.7M -> 22M; Spice_Model 4.7Meg -> 22Meg
- R2: value 2.7M -> 4.7M; Spice_Model 2.7Meg -> 4.7Meg
- R3: value 4M -> 4.7M; Spice_Model 4Meg -> 4.7Meg
- R8: Spice_Model 1meg -> 1Meg
- V1: Spice_Model dc 12 pulse(0 12 5m 1m 1m 15 30) -> dc 12 pulse(0 12 5m 1m 1m 20 30)
- renumbered R14 to R16, R15 to R17, R17 to R19, R18 to R20, R19 to R21, R20 to R22, R21 to R23
Connections:
- net GND: now also R15.2
- net Vc2: no longer R11.1
- net Vcc: now also R14.1
- net Vcomp2: now also R11.2
- net Vcomp3: now also R14.2, R15.1; no longer R11.2
- net Vgate: now also D6.1 (K), R11.1; no longer D6.2 (A)
- net at R9.1: now also D6.2 (A); no longer D6.1 (K)
Other:
- moved on the sheet: C3, C4, C5, D7, Q2, Q3, Q4, R12, R13, R16, R17, R18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
