File: kicad/GracefulPSU.kicad_sch (KiCad schematic)
At the start: 78 parts, among them J1 +12V in1, J10 +5Vu, J11 +5V, J12 0V, J2 +12V in2, J3 0v, J4 Conn_02x20, J5 Conn_02x20, J6 LED-, J7 Sw, J8 Sw, J9 LED+, Q1 CSD19505KCS, Q2 IRF7319, Q3 CSD19505KCS, U1 TLV9152, U2 LM22678TJ-ADJ

Commit message: Prep for release to github.
Parts:
- removed D12: 1N4148, Diode_THT:D_A-405_P7.62mm_Horizontal, symbol Device:D
- added B1: PSU_Board, my_extras:Buck Power Supply Board, symbol My_Extras:PSU_Board
- added D13, D6: 1N4148, my_extras:my_diode_7.62_h, symbol Device:D
- added R17: 1M, my_extras:my_resistor_6.3_2.5_10.16, symbol Device:R
- C10: value 27μF -> 56μF; footprint Capacitor_THT:CP_Radial_D5.0mm_P2.00mm -> Capacitor_SMD:CP_Elec_5x5.3
- C12: value 0.1μF -> 10nF
- C14: renamed from C13; value 1000μF -> 120μF; footprint Capacitor_THT:CP_Radial_D8.0mm_P2.50mm -> Capacitor_SMD:CP_Elec_6.3x5.9
- C8: footprint Capacitor_THT:CP_Radial_D5.0mm_P2.00mm -> my_extras:Capacitor_THT_HorizRadial_D5_P2_H12
- D1, D2, D3, D4, D5: footprint Diode_THT:D_A-405_P7.62mm_Horizontal -> my_extras:my_diode_7.62_h
- D10: renamed from D9; footprint Diode_THT:D_A-405_P7.62mm_Horizontal -> my_extras:my_diode_7.62_h
- D11: renamed from D10; value 6V8 -> 1V8; footprint Diode_THT:D_A-405_P7.62mm_Horizontal -> my_extras:my_diode_7.62_h
- D12: renamed from D11; footprint Diode_THT:D_A-405_P7.62mm_Horizontal -> my_extras:my_diode_7.62_h
- D14: renamed from D13; value SS54 -> SBRD 10200; footprint my_extras:DO-214AC -> Package_TO_SOT_SMD:TO-252-3_TabPin2
- D9: renamed from D8; footprint Diode_THT:D_A-405_P7.62mm_Horizontal -> my_extras:my_diode_7.62_h
- L1: value 6.8μH -> 3.9μH; footprint Inductor_SMD:L_Bourns-SRU1028_10.0x10.0mm -> my_extras:Shenzhen MWSA0604S
- Q1, Q3: footprint Package_TO_SOT_THT:TO-220-3_Vertical -> Package_TO_SOT_THT:TO-220-3_Horizontal_TabDown
- R1, R10, R12, R2, R25, R3, R4, R5, R6, R7, R8, R9: footprint Resistor_THT:R_Axial_DIN0207_L6.3mm_D2.5mm_P10.16mm_Horizontal -> my_extras:my_resistor_6.3_2.5_10.16
- R11: value 47M -> 22M; footprint Resistor_THT:R_Axial_DIN0207_L6.3mm_D2.5mm_P10.16mm_Horizontal -> my_extras:my_resistor_6.3_2.5_10.16
- R13: renamed from R15; value 1M -> 2M; footprint Resistor_THT:R_Axial_DIN0207_L6.3mm_D2.5mm_P10.16mm_Horizontal -> my_extras:my_resistor_6.3_2.5_10.16
- R14: renamed from R13; footprint Resistor_THT:R_Axial_DIN0207_L6.3mm_D2.5mm_P10.16mm_Horizontal -> my_extras:my_resistor_6.3_2.5_10.16
- R15: renamed from R14; footprint Resistor_THT:R_Axial_DIN0207_L6.3mm_D2.5mm_P10.16mm_Horizontal -> my_extras:my_resistor_6.3_2.5_10.16
- R16: renamed from R18; value 1M -> 2M; footprint Resistor_THT:R_Axial_DIN0207_L6.3mm_D2.5mm_P10.16mm_Horizontal -> my_extras:my_resistor_6.3_2.5_10.16
- R18: renamed from R16; value 330K -> 2M; footprint Resistor_THT:R_Axial_DIN0207_L6.3mm_D2.5mm_P10.16mm_Horizontal -> my_extras:my_resistor_6.3_2.5_10.16
- R19: renamed from R17; value 470K -> 1M; footprint Resistor_THT:R_Axial_DIN0207_L6.3mm_D2.5mm_P10.16mm_Horizontal -> my_extras:my_resistor_6.3_2.5_10.16
- R20: renamed from R19; value 4.7M -> 22M; footprint Resistor_THT:R_Axial_DIN0207_L6.3mm_D2.5mm_P10.16mm_Horizontal -> my_extras:my_resistor_6.3_2.5_10.16
- R21: renamed from R20; footprint Resistor_THT:R_Axial_DIN0207_L6.3mm_D2.5mm_P10.16mm_Horizontal -> my_extras:my_resistor_6.3_2.5_10.16
- R22: renamed from R21; footprint Resistor_THT:R_Axial_DIN0207_L6.3mm_D2.5mm_P10.16mm_Horizontal -> my_extras:my_resistor_6.3_2.5_10.16
- R23: renamed from R22; footprint Resistor_THT:R_Axial_DIN0207_L6.3mm_D2.5mm_P10.16mm_Horizontal -> my_extras:my_resistor_6.3_2.5_10.16
- R24: renamed from R23; footprint Resistor_THT:R_Axial_DIN0207_L6.3mm_D2.5mm_P10.16mm_Horizontal -> my_extras:my_resistor_6.3_2.5_10.16
- R26: renamed from R24; value 220K -> 270K; footprint Resistor_THT:R_Axial_DIN0207_L6.3mm_D2.5mm_P10.16mm_Horizontal -> my_extras:my_resistor_6.3_2.5_10.16
- R27: renamed from R26; footprint Resistor_THT:R_Axial_DIN0207_L6.3mm_D2.5mm_P10.16mm_Horizontal -> my_extras:my_resistor_6.3_2.5_10.16
- R28: renamed from R27; footprint Resistor_THT:R_Axial_DIN0207_L6.3mm_D2.5mm_P10.16mm_Horizontal -> my_extras:my_resistor_6.3_2.5_10.16
- R29: renamed from R28; footprint Resistor_THT:R_Axial_DIN0207_L6.3mm_D2.5mm_P10.16mm_Horizontal -> my_extras:my_resistor_6.3_2.5_10.16
- R30: renamed from R29; footprint Resistor_THT:R_Axial_DIN0207_L6.3mm_D2.5mm_P10.16mm_Horizontal -> my_extras:my_resistor_6.3_2.5_10.16
- R31: renamed from R30; footprint Resistor_THT:R_Axial_DIN0207_L6.3mm_D2.5mm_P10.16mm_Horizontal -> my_extras:my_resistor_6.3_2.5_10.16
- renumbered D6 to D7, D7 to D8
Connections:
- net +5V: now also B1.1 (+5V)
- net GND: now also B1.2 (Gnd), B1.4 (Vin-), R17.2
- net at C4.1, C5.1, D7.1 (K)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: now also R18.1; no longer R16.1
- net at C5.2, Q1.2 (D), R12.2: no longer R13.1
- net at C10.1, C11.1, C8.1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: now also B1.3 (Vin+), D13.2 (A); no longer R25.1
- net at D3.1 (K), D4.1 (K), J9.1 (Pin_1)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: now also R16.1, D6.2 (A); no longer C2.1, R18.1, R2.1
- net at D11.1 (K): now also R10.2, R11.2, R13.1, U1.7; no longer R14.1
- net at R13.2, R16.2: now also R25.1, U1.2 (-), R17.1; no longer R20.1, U1.3 (+)
- net at R18.2, R19.1: now also R20.1, U1.3 (+); no longer U1.2 (-)
- net at R25.2: now also D13.1 (K)
- new net: D11.2 (A), R14.1
- new net: C2.1, D6.1 (K), R2.1
Other:
- note added: "30 mΩ"
- note added: "Note 1: The PSU Board B1 is an optional component that replaces U2, L1, D14, C10, C11, C12, and C13. This can provide a higher current power supply at lower cost."
- note added: "Note 2: A push-to-make switch across J7 and J8 provides a power switch. With C5 fully charged and output power turned off, a momentary push of the switch turns output power on. With power on, a momentary push of the switch can be detected by a gpio (via JP3) allowing the SBC to turn off the power, either slowly via JP3 or more quickly via JP4. Tp force power-off, hold the switch on for several se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"
- note removed: "Note: A push-to-make switch across J7 and J8 provides a power switch. With C5 fully charged and output power turned off, a momentary push of the switch turns output power on. With power on, a momentary push of the switch can be detected by a gpio (via JP3) allowing the SBC to turn off the power, either slowly via JP3 or more quickly via JP4. Tp force power-off, hold the switch on for several seco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"
- moved on the sheet: C14, C2, C4, D11, D14, D3, D4, JP4, Q1, R12, R13, R14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

Commit message: Preparing for release to github.
Changed lines of the file:
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@@
   (title_block
     (title "Graceful SBC Power Supply")
+    (date "2024-03-27")
     (rev "3.0")
     (company "Bloodnok Marine")
@@
   )
   (text "Note 1: The PSU Board B1 is an optional component that replaces \nU2, L1, D14, C10, C11, C12, and C13.  This can provide a higher\ncurrent power supply at lower cost."
-    (at 179.07 145.415 0)
+    (at 192.405 147.32 0)
     (effects (font (size 1.27 1.27)) (justify left bottom))
   )
@@
   )
   (text "Note 2: A push-to-make switch across J7 and J8 provides a power switch.\nWith C5 fully charged and output power turned off, a momentary push\nof the switch turns output power on.\n\nWith power on, a momentary push of the switch can be detected by \na gpio (via JP3) allowing the SBC to turn off the power, either\nslowly via JP3 or more quickly via JP4.\n\nTp force power-off, hold the switch on for several seconds."
-    (at 179.07 167.64 0)
+    (at 192.405 169.545 0)
     (effects (font (size 1.27 1.27)) (justify left bottom))
   )
@@
     (effects (font (size 1.27 1.27)) (justify left bottom))
   )
+  (text "*" (at 175.895 131.445 0)
+    (effects (font (size 1.27 1.27)) (justify left bottom))
+  )
   (text "30 mΩ" (at 250.825 113.03 0)
     (effects (font (size 0.7 0.7)) (justify left bottom))
@@
     (effects (font (size 1.27 1.27)) (justify left bottom))
   )
+  (text "*" (at 192.405 127.635 0)
+    (effects (font (size 1.27 1.27)) (justify left bottom))
+  )
   (text "*" (at 152.4 64.77 0)
     (effects (font (size 1.27 1.27)) (justify left bottom))
@@
   (symbol (lib_id "Device:R") (at 149.86 105.41 270) (unit 1)
     (in_bom yes) (on_board yes)
-    (property "Reference" "R22" (id 0) (at 149.86 100.4275 90))
+    (property "Reference" "R22" (id 0) (at 147.955 100.965 90))
     (property "Value" "1K" (id 1) (at 149.86 103.2026 90))
     (property "Footprint" "my_extras:my_resistor_6.3_2.5_10.16" (id 2) (at 149.86 103.632 90)
